File: Hardware/SparkFun_Red_Vision_Camera_Board_HM01B0.kicad_sch (KiCad schematic)
At the start: 46 parts, among them J1 Conn_01x09, J2 Conn_01x09, J3 Conn_01x09, J4 HM01B0, Q1 RE1C002UNTCL, Q2 RE1C002UNTCL, Q3 RE1C002UNTCL, Q4 RE1C002UNTCL, U1 HM01B0, U2 RT9080-2.8V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

Commit message: Update libraries
Parts:
- J4: footprint lcd-tft:Socket_2x12_0.4mm-pitch_5055502420 -> SparkFun-Connector:FPC_2x12-1MP_P0.4mm; symbol HM0360:Conn_2x15_Camera_HM01B0 -> SparkFun-Camera:Camera_HM01B0_Connector
- U1: symbol HM0360:HM01B0-ANA-00FT870 -> SparkFun-Camera:Camera_HM01B0_Outline
Changed lines of the file:
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@@
 (kicad_sch
-	(version 20231120)
+	(version 20250114)
 	(generator "eeschema")
-	(generator_version "8.0")
+	(generator_version "9.0")
 	(paper "USLetter")
 	(title_block
@@
 		(comment 1 "Designed by: Dryw Wade")
 	)
+	(text "Connect XCLK to only 1 at\na time, otherwise undefined\nbehavior or damage may occur"
+		(exclude_from_sim no)
+		(at 250.19 80.01 0)
+		(effects
+			(font
+				(size 1.27 1.27)
+			)
+		)
+	)
+	(text "I2C Address: 0x24"
+		(exclude_from_sim no)
+		(at 49.53 82.55 0)
+		(effects
+			(font
+				(size 1.27 1.27)
+			)
+		)
+	)
+	(text "24MHz Oscillator"
+		(exclude_from_sim no)
+		(at 238.76 87.63 0)
+		(effects
+			(font
+				(size 1.27 1.27)
+			)
+		)
+	)
+	(text "Solder OSC_DIS jumper\nto disable oscillator"
+		(exclude_from_sim no)
+		(at 199.39 114.3 0)
+		(effects
+			(font
+				(size 1.27 1.27)
+			)
+		)
+	)
+	(text "Jumper Setting"
+		(exclude_from_sim no)
+		(at 259.08 85.09 0)
+		(effects
+			(font
+				(size 1.27 1.27)
+			)
+		)
+	)
+	(text "Cut I2C jumper to\nremove pullup resistors"
+		(exclude_from_sim no)
+		(at 223.52 147.32 0)
+		(effects
+			(font
+				(size 1.27 1.27)
+			)
+		)
+	)
+	(text "Camera - HM01B0"
+		(exclude_from_sim no)
+		(at 52.07 15.24 0)
+		(effects
+			(font
+				(size 2.54 2.54)
+			)
+		)
+	)
+	(text "Clock Source"
+		(exclude_from_sim no)
+		(at 238.76 85.09 0)
+		(effects
+			(font
+				(size 1.27 1.27)
+			)
+		)
+	)
+	(text "Headers"
+		(exclude_from_sim no)
+		(at 215.9 15.24 0)
+		(effects
+			(font
+				(size 2.54 2.54)
+			)
+		)
+	)
+	(text "I2C Pullup Resistors"
+		(exclude_from_sim no)
+		(at 223.52 123.19 0)
+		(effects
+			(font
+				(size 2.54 2.54)
+			)
+		)
+	)
+	(text "OSC (default)"
+		(exclude_from_sim no)
+		(at 259.08 87.63 0)
+		(effects
+			(font
+				(size 1.27 1.27)
+			)
+		)
+	)
+	(text "Voltage Regulator - RT9080"
+		(exclude_from_sim no)
+		(at 88.9 123.19 0)
+		(effects
+			(font
+				(size 2.54 2.54)
+			)
+		)
+	)
+	(text "GND"
+		(exclude_from_sim no)
+		(at 259.08 92.71 0)
+		(effects
+			(font
+				(size 1.27 1.27)
+			)
+		)
+	)
+	(text "Cut PWR jumper to\ndisable power LED"
+		(exclude_from_sim no)
+		(at 173.99 129.54 0)
+		(effects
+			(font
+				(size 1.27 1.27)
+			)
+		)
+	)
+	(text "Power LED"
+		(exclude_from_sim no)
+		(at 172.72 123.19 0)
+		(effects
+			(font
+				(size 2.54 2.54)
+			)
+		)
+	)
+	(text "XCLK Generator and Selection"
+		(exclude_from_sim no)
+		(at 215.9 74.93 0)
+		(effects
+			(font
+				(size 2.54 2.54)
+			)
+		)
+	)
+	(text "I2C Level Shifters "
+		(exclude_from_sim no)
+		(at 127 15.24 0)
+		(effects
+			(font
+				(size 2.54 2.54)
+			)
+		)
+	)
+	(text "XCLK PTH Pad"
+		(exclude_from_sim no)
+		(at 238.76 90.17 0)
+		(effects
+			(font
+				(size 1.27 1.27)
+			)
+		)
+	)
+	(text "Internal 48MHz Oscillator"
+		(exclude_from_sim no)
+		(at 238.76 92.71 0)
+		(effects
+			(font
+				(size 1.27 1.27)
+			)
+		)
+	)
+	(text "PAD"
+		(exclude_from_sim no)
+		(at 259.08 90.17 0)
+		(effects
+			(font
+				(size 1.27 1.27)
+			)
+		)
+	)
 	(junction
 		(at 86.36 149.86)
@@
 		)
 	)
-	(text "Connect XCLK to only 1 at\na time, otherwise undefined\nbehavior or damage may occur"
-		(exclude_from_sim no)
-		(at 250.19 80.01 0)
-		(effects
-			(font
-				(size 1.27 1.27)
-			)
-		)
-	)
-	(text "I2C Address: 0x24"
-		(exclude_from_sim no)
-		(at 49.53 82.55 0)
-		(effects
-			(font
-				(size 1.27 1.27)
-			)
-		)
-	)
-	(text "24MHz Oscillator"
-		(exclude_from_sim no)
-		(at 238.76 87.63 0)
-		(effects
-			(font
-				(size 1.27 1.27)
-			)
-		)
-	)
-	(text "Solder OSC_DIS jumper\nto disable oscillator"
-		(exclude_from_sim no)
-		(at 199.39 114.3 0)
-		(effects
-			(font
-				(size 1.27 1.27)
-			)
-		)
-	)
-	(text "Jumper Setting"
-		(exclude_from_sim no)
-		(at 259.08 85.09 0)
-		(effects
-			(font
-				(size 1.27 1.27)
-			)
-		)
-	)
-	(text "Cut I2C jumper to\nremove pullup resistors"
-		(exclude_from_sim no)
-		(at 223.52 147.32 0)
-		(effects
-			(font
-				(size 1.27 1.27)
-			)
-		)
-	)
-	(text "Camera - HM01B0"
-		(exclude_from_sim no)
-		(at 52.07 15.24 0)
-		(effects
-			(font
-				(size 2.54 2.54)
-			)
-		)
-	)
-	(text "Clock Source"
-		(exclude_from_sim no)
-		(at 238.76 85.09 0)
-		(effects
-			(font
-				(size 1.27 1.27)
-			)
-		)
-	)
-	(text "Headers"
-		(exclude_from_sim no)
-		(at 215.9 15.24 0)
-		(effects
-			(font
-				(size 2.54 2.54)
-			)
-		)
-	)
-	(text "I2C Pullup Resistors"
-		(exclude_from_sim no)
-		(at 223.52 123.19 0)
-		(effects
-			(font
-				(size 2.54 2.54)
-			)
-		)
-	)
-	(text "OSC (default)"
-		(exclude_from_sim no)
-		(at 259.08 87.63 0)
-		(effects
-			(font
-				(size 1.27 1.27)
-			)
-		)
-	)
-	(text "Voltage Regulator - RT9080"
-		(exclude_from_sim no)
-		(at 88.9 123.19 0)
-		(effects
-			(font
-				(size 2.54 2.54)
-			)
-		)
-	)
-	(text "GND"
-		(exclude_from_sim no)
-		(at 259.08 92.71 0)
-		(effects
-			(font
-				(size 1.27 1.27)
-			)
-		)
-	)
-	(text "Cut PWR jumper to\ndisable power LED"
-		(exclude_from_sim no)
-		(at 173.99 129.54 0)
-		(effects
-			(font
-				(size 1.27 1.27)
-			)
-		)
-	)
-	(text "Power LED"
-		(exclude_from_sim no)
-		(at 172.72 123.19 0)
-		(effects
-			(font
-				(size 2.54 2.54)
-			)
-		)
-	)
-	(text "XCLK Generator and Selection"
-		(exclude_from_sim no)
-		(at 215.9 74.93 0)
-		(effects
-			(font
-				(size 2.54 2.54)
-			)
-		)
-	)
-	(text "I2C Level Shifters "
-		(exclude_from_sim no)
-		(at 127 15.24 0)
-		(effects
-			(font
-				(size 2.54 2.54)
-			)
-		)
-	)
-	(text "XCLK PTH Pad"
-		(exclude_from_sim no)
-		(at 238.76 90.17 0)
-		(effects
-			(font
-				(size 1.27 1.27)
-			)
-		)
-	)
-	(text "Internal 48MHz Oscillator"
-		(exclude_from_sim no)
-		(at 238.76 92.71 0)
-		(effects
-			(font
-				(size 1.27 1.27)
-			)
-		)
-	)
-	(text "PAD"
-		(exclude_from_sim no)
-		(at 259.08 90.17 0)
-		(effects
-			(font
-				(size 1.27 1.27)
-			)
-		)
-	)
 	(global_label "CAM_VS"
 		(shape input)
@@
 	)
 	(symbol
-		(lib_id "HM0360:HM01B0-ANA-00FT870")
+		(lib_id "SparkFun-Camera:Camera_HM01B0_Outline")
 		(at 49.53 72.39 0)
 		(unit 1)
@@
 			)
 		)
-		(property "Datasheet" "https://cdn.sparkfun.com/datasheets/BreakoutBoards/BSS138.pdf"
+		(property "Datasheet" "https://fscdn.rohm.com/en/products/databook/datasheet/discrete/transistor/mosfet/re1c002untcl-e.pdf"
 			(at 114.3 58.42 0)
 			(effects
@@
 			)
 		)
-		(property "Datasheet" "https://cdn.sparkfun.com/datasheets/BreakoutBoards/BSS138.pdf"
+		(property "Datasheet" "https://fscdn.rohm.com/en/products/databook/datasheet/discrete/transistor/mosfet/re1c002untcl-e.pdf"
 			(at 114.3 93.98 0)
 			(effects
@@
 			)
 		)
-		(property "Datasheet" "https://cdn.sparkfun.com/datasheets/BreakoutBoards/BSS138.pdf"
+		(property "Datasheet" "https://fscdn.rohm.com/en/products/databook/datasheet/discrete/transistor/mosfet/re1c002untcl-e.pdf"
 			(at 40.64 170.18 0)
 			(effects
@@
 	)
 	(symbol
-		(lib_id "HM0360:Conn_2x15_Camera_HM01B0")
+		(lib_id "SparkFun-Camera:Camera_HM01B0_Connector")
 		(at 49.53 52.07 0)
 		(unit 1)
@@
 			)
 		)
-		(property "Footprint" "lcd-tft:Socket_2x12_0.4mm-pitch_5055502420"
+		(property "Footprint" "SparkFun-Connector:FPC_2x12-1MP_P0.4mm"
 			(at 49.53 76.2 0)
 			(effects
@@
 			)
 		)
-		(property "Datasheet" "https://cdn.sparkfun.com/datasheets/BreakoutBoards/BSS138.pdf"
+		(property "Datasheet" "https://fscdn.rohm.com/en/products/databook/datasheet/discrete/transistor/mosfet/re1c002untcl-e.pdf"
 			(at 83.82 170.18 0)
 			(effects
@@
 		)
 	)
+	(embedded_fonts no)
 )
